File: kicad/protoboard-40x60mm-gndplane/protoboard-40x60mm-gndplane.kicad_pcb (KiCad board)
At the start: 2 copper layers, 60 x 40 mm, 1057 parts

Commit message: Update 40x60mm gndplane PCB with new tolerances
Parts:
- REF** (x280): footprint modules:tht-0.8-thin-bottom -> MeineBib:Proto_Advanced_Pin_Gndplane
